File: QCPU/qcpu_eval_board/qcpu_eval_board.kicad_sch (KiCad schematic)
At the start: 20 parts, among them J1 Conn_01x12, J2 Conn_01x12, U1 gfmpw1-multi, U2 74HC32, U3 W25Q32JVSS, U4 74HC74, U5 74LS08, X1 CXO_DIP8

Commit message: QCPU eval board PCB design
Parts:
- added C2, C3, C4, C5: 100nF, Capacitor_THT:C_Disc_D3.8mm_W2.6mm_P2.50mm, symbol Device:C
- added D1, D2: LED, LED_THT:LED_D5.0mm, symbol Device:LED
- added J3, J4, J6: Conn_01x08, Connector_PinHeader_2.54mm:PinHeader_1x08_P2.54mm_Vertical, symbol Connector_Generic:Conn_01x08
- added J5: Conn_01x06, Connector_PinSocket_2.54mm:PinSocket_1x06_P2.54mm_Vertical, symbol Connector_Generic:Conn_01x06
- added J7: Screw_Terminal_01x02, TerminalBlock:TerminalBlock_bornier-2_P5.08mm, symbol Connector:Screw_Terminal_01x02
- added R12, R13: 1K, Resistor_THT:R_Axial_DIN0204_L3.6mm_D1.6mm_P7.62mm_Horizontal, symbol Device:R
- U2, U4, U5: footprint (none) -> Package_DIP:DIP-14_W7.62mm
- U3: footprint Package_SO:SOIC-8_5.23x5.23mm_P1.27mm -> Package_DIP:DIP-8_W7.62mm
Connections:
- net +3V3: now also C4.1, C5.1
- net +5V: now also C2.1, C3.1, J7.2 (Pin_2)
- net FREQ: now also J6.3 (Pin_3)
- net GND: now also C2.2, C3.2, C4.2, C5.2, J5.2 (Pin_2), J7.1 (Pin_1), R12.2, R13.2
- net PA0: now also D1.2 (A), J3.1 (Pin_1)
- net PA1: now also D2.2 (A), J3.2 (Pin_2)
- net PA2: now also J3.3 (Pin_3)
- net PA3: now also J3.4 (Pin_4)
- net PA4: now also J3.5 (Pin_5)
- net PA5: now also J3.6 (Pin_6)
- net PA6: now also J3.7 (Pin_7)
- net PA7: now also J3.8 (Pin_8)
- net PB0: now also J4.1 (Pin_1)
- net PB1: now also J4.2 (Pin_2)
- net PB2: now also J4.3 (Pin_3)
- net PB3: now also J4.4 (Pin_4)
- net PB4: now also J4.5 (Pin_5)
- net PB5: now also J4.6 (Pin_6)
- net PB6: now also J4.7 (Pin_7)
- net PB7: now also J4.8 (Pin_8)
- net PWM: now also J6.2 (Pin_2)
- net RXD: now also J5.3 (Pin_3)
- net SCLK: now also J6.4 (Pin_4)
- net SCLK_3v3: now also J6.8 (Pin_8)
- net SDI: now also J6.6 (Pin_6)
- net SDO: now also J6.5 (Pin_5)
- net SDO_3v3: now also J6.7 (Pin_7)
- net TXD: now also J5.4 (Pin_4)
- net ~{INT}: now also J6.1 (Pin_1)
- new net: D1.1 (K), R12.1
- new net: D2.1 (K), R13.1
- no-connect marks 8 -> 11
