File: TholinRISCV/gfmpw1-tholin-riscv/gfmpw1-tholin-riscv.kicad_pcb (KiCad board)
At the start: 4 copper layers, 97.5 x 81.8 mm, 35 parts, among them J1 Screw_Terminal_01x02, J2 Conn_01x06, J3 Micro_SD_Card, J4 Conn_01x06, J5 Conn_02x05_Counter_Clockwise, J6 Conn_01x03, SW1 SW_Push, SW2 SW_Push, U1 gfmpw1-multi, U10 74LS08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

Commit message: Minor tweaks, make QCPU work
Parts:
- added C6: 22pF, Capacitor_THT:C_Disc_D3.8mm_W2.6mm_P2.50mm, F.Cu at (207.8, 103.9)
- added R6: 10K, Resistor_THT:R_Axial_DIN0204_L3.6mm_D1.6mm_P7.62mm_Horizontal, F.Cu at (225.0, 93.7)
Routing:
- net Net-(J3-DAT0): track 37.1 -> 52.9 mm
- net SCLK: track 93.5 -> 98.0 mm
- net +3V3: track 153.0 -> 155.3 mm
