File: TholinRISCV/gfmpw1-tholin-riscv/gfmpw1-tholin-riscv.kicad_sch (KiCad schematic)
At the start: 33 parts, among them J1 Screw_Terminal_01x02, J2 Conn_01x06, J3 Micro_SD_Card, J4 Conn_01x06, J5 Conn_02x05_Counter_Clockwise, J6 Conn_01x03, SW1 SW_Push, SW2 SW_Push, U1 gfmpw1-multi, U10 74LS08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

Commit message: Minor tweaks, make QCPU work
Parts:
- added C6: 22pF, Capacitor_THT:C_Disc_D3.8mm_W2.6mm_P2.50mm, symbol Device:C
- added R6: 10K, Resistor_THT:R_Axial_DIN0204_L3.6mm_D1.6mm_P7.62mm_Horizontal, symbol Device:R
Connections:
- net +3V3: now also R6.1
- net GND: now also C6.2
- net SCLK: now also C6.1
- net at J3.7 (DAT0), J5.4 (Pin_4), U11.2 (A): now also R6.2
